File: motor-logger/motor-logger.kicad_sch (KiCad schematic)
At the start: 56 parts, among them J1 Conn_01x02_Pin, J2 Conn_01x02_Pin, J3 Conn_01x02_Pin, J4 Conn_01x02_Pin, J5 ST7920 128X64 LCD Display, Q1 BSS138, Q2 BSS138, SW1 SW_Push, SW2 SW_Push, U1 MCP6004, U2 AMS1117-3.3, U3 CH340C, U5 AMS1117-3.3

Commit message: -
Parts:
- C1: LCSC (none) -> C15850
- C2: renamed from C3; LCSC (none) -> C15850
- C5: renamed from C4; LCSC (none) -> C15850
- C6: renamed from C5; LCSC (none) -> C49678
- C9: renamed from C2; LCSC (none) -> C15850
- J1: footprint (none) -> Connector_JST:JST_XH_B2B-XH-A_1x02_P2.50mm_Vertical
- J2: renamed from J3; footprint (none) -> Connector_JST:JST_XH_B2B-XH-A_1x02_P2.50mm_Vertical
- J3: renamed from J2; footprint (none) -> Connector_JST:JST_XH_B2B-XH-A_1x02_P2.50mm_Vertical
- J4: footprint (none) -> TerminalBlock:TerminalBlock_MaiXu_MX126-5.0-02P_1x02_P5.00mm
- R1: footprint (none) -> Resistor_SMD:R_0603_1608Metric_Pad0.98x0.95mm_HandSolder; LCSC (none) -> C21190
- R11: renamed from R9; value 1K -> 1k
- R12: renamed from R8; value 1K -> 1k
- R13: value 1K -> 1k
- R14: renamed from R11; value 1K -> 1k
- R2: renamed from R5; footprint (none) -> Resistor_SMD:R_0603_1608Metric_Pad0.98x0.95mm_HandSolder; LCSC (none) -> C21190
- R3: renamed from R2; footprint (none) -> Resistor_SMD:R_0603_1608Metric_Pad0.98x0.95mm_HandSolder; LCSC (none) -> C105588
- R4: renamed from R6; footprint (none) -> Resistor_SMD:R_0603_1608Metric_Pad0.98x0.95mm_HandSolder; LCSC (none) -> C105588
- R5: renamed from R10; value 1K -> 1k
- R6: renamed from R14; value 1K -> 1k
- R7: renamed from R3; footprint (none) -> Resistor_SMD:R_0603_1608Metric_Pad0.98x0.95mm_HandSolder; LCSC (none) -> C21190
- R8: renamed from R4; footprint (none) -> Resistor_SMD:R_0603_1608Metric_Pad0.98x0.95mm_HandSolder; LCSC (none) -> C105588
- U5: renamed from U4; value ~ -> ESP32_S2
- USB1: value ~ -> USB_TYPE_C
- renumbered C8 to C10, C9 to C11, C10 to C12, C11 to C13, C12 to C14, C13 to C15, C14 to C16, C6 to C3, C15 to C4, C16 to C8, D9 to D2, D2 to D5, JP2 to JP1, JP1 to JP2, JP4 to JP3, JP3 to JP4, R8 to R10, R7 to R9, U5 to U3, U3 to U4

Commit message: -
Parts:
- added C11, C12, C13, C9: 22uF, Capacitor_SMD:C_0603_1608Metric, symbol Device:C
- added C20, C21, C22, C23: 0.1uF, Capacitor_SMD:C_0805_2012Metric_Pad1.18x1.45mm_HandSolder, symbol Device:C
- added D3, D4: LED, LED_SMD:LED_0805_2012Metric_Pad1.15x1.40mm_HandSolder, symbol Device:LED
- added JP10, JP3, JP4, JP7, JP8, JP9: SolderJumper_2_Open, Jumper:SolderJumper-2_P1.3mm_Open_RoundedPad1.0x1.5mm, symbol Jumper:SolderJumper_2_Open
- added R10, R16, R17, R18, R19, R8: 1k, Resistor_SMD:R_0603_1608Metric_Pad0.98x0.95mm_HandSolder, symbol Device:R
- added SW2, SW3, SW4, SW5: SW_Push, Button_Switch_THT:SW_PUSH_6mm_H9.5mm, symbol Switch:SW_Push
- added U4, U5: AMS1117-3.3, Package_TO_SOT_SMD:SOT-223-3_TabPin2, symbol Regulator_Linear:AMS1117-3.3
- J5: footprint Connector_PinHeader_2.54mm:PinHeader_1x20_P2.54mm_Vertical -> footprint_motor:LCD-TH_HS12864-15C
- R1, R2, R7: footprint Resistor_SMD:R_0603_1608Metric_Pad0.98x0.95mm_HandSolder -> Resistor_SMD:R_0805_2012Metric_Pad1.20x1.40mm_HandSolder
- R4: renamed from R3; footprint Resistor_SMD:R_0603_1608Metric_Pad0.98x0.95mm_HandSolder -> Resistor_SMD:R_0805_2012Metric_Pad1.20x1.40mm_HandSolder
- R9: renamed from R8; footprint Resistor_SMD:R_0603_1608Metric_Pad0.98x0.95mm_HandSolder -> Resistor_SMD:R_0805_2012Metric_Pad1.20x1.40mm_HandSolder
- U7: renamed from U5; value ESP32_S2 -> ESP32_S3
- renumbered C9 to C10, C10 to C14, C11 to C15, C12 to C16, C13 to C17, C14 to C18, C15 to C19, C16 to C24, C4 to C3, C8 to C4, C3 to C5, C5 to C6, C6 to C7, C7 to C8, D2 to D1, D1 to D2, D3 to D5, D4 to D6, D5 to D7, JP2 to JP1, JP5 to JP11, JP1 to JP2, JP3 to JP5, JP4 to JP6, R9 to R11, R10 to R12, R11 to R13, R12 to R14, R13 to R15, R14 to R20, R6 to R3, R4 to R5, R5 to R6, SW2 to SW6, U3 to U1, U1 to U2, U2 to U3, U4 to U6
Connections:
- net +3.3V: now also JP7.2 (B), JP9.2 (B), R16.1, R17.1, R18.1, R19.1
- net +3V3: no longer C4.2, JP1.1 (A), R1.1, R2.1, R7.1, U1.2 (VO)
- net +5V: now also C12.2, C9.2, JP10.2 (B), JP8.2 (B), U4.3 (VI), U5.3 (VI); no longer J5.2 (Pin_2), RV1.1
- net GND: now also C11.1, C12.1, C13.1, C20.1, C21.1, C22.1, C23.1, C9.1, R10.2, R8.2, SW2.1, SW3.1, SW4.1, SW5.1, U4.1 (GND), U5.1 (GND)
- net PHASE1: now reaches U7.10 (IO17)
- net PHASE1: now also C22.2, R18.2, SW4.2
- net PHASE2: now reaches U7.11 (IO18)
- net PHASE2: now also C23.2, R19.2, SW5.2
- net PHASE3: now reaches U7.12 (IO8)
- net PHASE3: now also C20.2, R16.2, SW2.2
- net CAL: now reaches U7.9 (IO16)
- net CAL: now also C21.2, R17.2, SW3.2
- new net: JP10.1 (A), JP9.1 (A), RV1.1
- new net: J5.2 (Pin_2), JP7.1 (A), JP8.1 (A)
- new net: D4.1 (K), R10.1
- new net: D4.2 (A), JP4.2 (B)
- new net: D3.2 (A), JP3.2 (B)
- new net: D3.1 (K), R8.1
- new net +3V3A: C4.2, JP1.1 (A), R1.1, U1.2 (VO)
- new net +3V3B: C11.2, JP3.1 (A), R7.1, U4.2 (VO)
- new net +3V3C: C13.2, JP4.1 (A), R2.1, U5.2 (VO)
- no-connect marks 49 -> 45
Other:
- moved on the sheet: C3, C4, C5, C8, D1, D2, JP1, JP2, R3, R6, U1, U3

Commit message: -
Parts:
- added JP12: SolderJumper_2_Open, Jumper:SolderJumper-2_P1.3mm_Open_RoundedPad1.0x1.5mm, symbol Jumper:SolderJumper_2_Open
- R5: footprint Resistor_SMD:R_0603_1608Metric_Pad0.98x0.95mm_HandSolder -> Resistor_SMD:R_0805_2012Metric_Pad1.20x1.40mm_HandSolder
Connections:
- net +3V3 is gone; now on net +3.3V: JP6.2 (B)
- net +5V: now also JP12.2 (B)
- net at J5.19 (Pin_19), JP6.1 (A): now also JP12.1 (A)
Other:
- moved on the sheet: JP6

Commit message: -
Parts:
- removed J1, J2, J3: Conn_01x02_Pin, Connector_JST:JST_XH_B2B-XH-A_1x02_P2.50mm_Vertical, symbol Connector:Conn_01x02_Pin
- added J1, J10, J2: Barrel_Jack_MountingPin, Connector_BarrelJack:BarrelJack_GCT_DCJ200-10-A_Horizontal, symbol Connector:Barrel_Jack_MountingPin
Connections:
- net at R2.2, U2.5 (+): now also J2.1
- net at R1.2, U2.3 (+): now also J10.1
- net at R7.2, U2.10 (+): now also J1.1
- net at C10.1: now also J1.2
- net at C2.1: now also J2.2
- net at C1.1: now also J10.2
- no-connect marks 45 -> 48
