File: motor-logger/motor-logger.kicad_pcb (KiCad board)
At the start: 2 copper layers, 106.8 x 73.5 mm, 84 parts, among them J1 Conn_01x02_Pin, J2 Conn_01x02_Pin, J3 Conn_01x02_Pin, J4 Conn_01x02_Pin, J5 ST7920 128X64 LCD Display, Q1 BSS138, Q2 BSS138, SW1 SW_Push, SW2 SW_Push, SW3 SW_Push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

Commit message: -
Parts:
- added JP12: SolderJumper_2_Open, Jumper:SolderJumper-2_P1.3mm_Open_RoundedPad1.0x1.5mm, B.Cu at (128.3, 102.6)
- added REF**: MountingHole_3.2mm_M3_DIN965_Pad_TopBottom, MountingHole:MountingHole_3.2mm_M3_DIN965_Pad_TopBottom, F.Cu at (213.2, 120.5)
- added REF**: MountingHole_3.2mm_M3_DIN965_Pad_TopBottom, MountingHole:MountingHole_3.2mm_M3_DIN965_Pad_TopBottom, F.Cu at (100.5, 39.2)
- added REF**: MountingHole_3.2mm_M3_DIN965_Pad_TopBottom, MountingHole:MountingHole_3.2mm_M3_DIN965_Pad_TopBottom, F.Cu at (213.2, 39.2)
- added REF**: MountingHole_3.2mm_M3_DIN965_Pad_TopBottom, MountingHole:MountingHole_3.2mm_M3_DIN965_Pad_TopBottom, F.Cu at (100.5, 120.5)
- JP1, JP10, JP11, JP2, JP3, JP4, JP5, JP6, JP7, JP8, JP9, RV1: moved to B.Cu
- R5: footprint Resistor_SMD:R_0603_1608Metric_Pad0.98x0.95mm_HandSolder -> Resistor_SMD:R_0805_2012Metric_Pad1.20x1.40mm_HandSolder
- moved J4 209.5 mm to (101.9, 110.0), turned to 90 degrees
- moved Q1 201.0 mm to (120.2, 76.5)
- moved Q2 200.9 mm to (120.2, 83.1)
- moved R13 189.0 mm to (102.9, 72.7), turned to 180 degrees
- moved R6 188.5 mm to (101.2, 57.2), turned to -90 degrees
- moved R14 188.2 mm to (102.9, 87.1), turned to 180 degrees
- moved U6 187.6 mm to (114.2, 79.8)
- moved JP2 186.6 mm to (101.2, 55.3), turned to 90 degrees
- moved R12 184.3 mm to (106.9, 78.2), turned to 90 degrees
- moved R11 184.1 mm to (106.9, 81.5), turned to -90 degrees
- moved SW1 171.3 mm to (140.9, 55.7), turned to 90 degrees
- moved USB1 170.2 mm to (100.8, 79.8), turned to -90 degrees
- moved JP6 167.3 mm to (125.8, 102.6), turned to 90 degrees
- moved RV1 162.3 mm to (165.2, 102.5), turned to 90 degrees
- moved JP5 161.7 mm to (132.0, 102.6), turned to 90 degrees
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Connections:
- JP6 pad 2: +3V3 -> +3.3V
Routing:
- net +3.3V: track 0.00 -> 396.3 mm, vias 0 -> 10
- net +5V: track 0.00 -> 297.8 mm, vias 0 -> 4
- net PHASE3: track 0.00 -> 96.5 mm
- net ESP_TX: track 0.00 -> 90.1 mm, vias 0 -> 2
- net PHASE2: track 0.00 -> 85.5 mm
- net ESP_RX: track 0.00 -> 84.4 mm, vias 0 -> 2
- net PHASE1: track 0.00 -> 75.6 mm
- net CAL: track 0.00 -> 70.9 mm
- net GND: track 0.00 -> 68.7 mm, vias 0 -> 43
- net ESP_I0: track 0.00 -> 66.8 mm, vias 0 -> 2
- net Net-(J3-Pin_1): track 0.00 -> 61.4 mm, vias 0 -> 2
- net RST_LCD: track 0.00 -> 59.5 mm, vias 0 -> 1
- net ESP_EN: track 0.00 -> 57.7 mm, vias 0 -> 2
- net SPI_CS: track 0.00 -> 51.1 mm, vias 0 -> 1
- net SPI_MOSI: track 0.00 -> 47.4 mm, vias 0 -> 1
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- added copper zone on B.Cu, net GND
- added copper zone on F.Cu, net GND
Other:
- board size 106.8 x 73.5 mm -> 119.2 x 87.8 mm

Commit message: -
Parts:
- moved J4 4.78 mm to (102.1, 105.2), turned to -90 degrees
Routing:
- net GND: track 68.7 -> 81.2 mm, vias 43 -> 50
- net Net-(D7-K): track 0.00 -> 6.65 mm
- net Net-(J5-Pin_17): track 0.00 -> 4.51 mm
- net +5V: track 297.8 -> 293.4 mm
- net Net-(D7-A): track 0.00 -> 4.28 mm, vias 0 -> 1

Commit message: -
Parts:
- moved U7 0.42 mm to (156.9, 56.5)
- moved D5 0.15 mm to (99.4, 72.7)
- moved D6 0.11 mm to (99.3, 87.1)
- moved R13 0.08 mm to (103.0, 72.7)
Routing:
- net GND: track 81.2 -> 101.9 mm, vias 50 -> 60
- net Net-(U2C--): track 29.5 -> 27.6 mm
- net Net-(JP11-A): track 11.3 -> 12.0 mm
- net ESP_TX: track 90.1 -> 89.5 mm
Other:
- board text added: "*"
- board text added: "3V3_LED"
- board text added: "3V3_ON"
- board text added: "5V"
- board text added: "BLA_3V3"
- board text added: "BLA_5V"
- board text added: "BOOT0"
- board text added: "CAL/START"
- board text added: "ESP_LED"
- board text added: "GND"
- board text added: "LCD_3V3"
- board text added: "LCD_5V"
- board text added: "LED_P1"
- board text added: "LED_P2"
- board text added: "LED_P3"
- board text added: "PROBE1"
- board text added: "PROBE2"
- board text added: "PROBE3"
- board text added: "RESET"
- board text added: "RST_LCD"
- board text added: "RV_3V3"
- board text added: "RV_5V"
- board text added: "RX"
- board text added: "TX"
- board text added: "VIN"

Commit message: -
Parts:
- removed J3: Conn_01x02_Pin, Connector_JST:JST_XH_B2B-XH-A_1x02_P2.50mm_Vertical
- added J10: Barrel_Jack_MountingPin, Connector_BarrelJack:BarrelJack_GCT_DCJ200-10-A_Horizontal, F.Cu at (209.5, 61.8)
- J1, J2: value Conn_01x02_Pin -> Barrel_Jack_MountingPin; footprint Connector_JST:JST_XH_B2B-XH-A_1x02_P2.50mm_Vertical -> Connector_BarrelJack:BarrelJack_GCT_DCJ200-10-A_Horizontal
- moved SW6 75.3 mm to (103.0, 94.0), turned to 180 degrees
- moved SW1 39.2 mm to (103.0, 65.7), turned to 0 degrees
- moved J1 34.9 mm to (209.5, 98.0)
- moved C20 18.4 mm to (193.4, 112.8)
- moved R16 18.4 mm to (197.0, 112.8)
- moved SW2 18.2 mm to (198.0, 119.8)
- moved C21 14.5 mm to (121.2, 112.7)
- moved R17 14.5 mm to (124.9, 112.7)
- moved SW3 14.4 mm to (126.0, 119.8)
- moved SW5 7.35 mm to (174.0, 119.8)
- moved C23 7.30 mm to (169.2, 112.7)
- moved R19 7.30 mm to (172.9, 112.7)
- moved REF** 3.83 mm to (217.1, 120.5)
- moved REF** 3.83 mm to (217.1, 39.2)
- moved C22 3.60 mm to (145.1, 112.8)
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Connections:
- C1 pad 1: Net-(J1-Pin_2) -> Net-(C1-Pad1)
- C10 pad 1: Net-(J3-Pin_2) -> Net-(C10-Pad1)
- J1 pad 1: Net-(J1-Pin_1) -> Net-(U2C-+)
- J1 pad 2: Net-(J1-Pin_2) -> Net-(C10-Pad1)
- R1 pad 2: Net-(J1-Pin_1) -> Net-(U2A-+)
- R7 pad 2: Net-(J3-Pin_1) -> Net-(U2C-+)
- U2 pad 10: Net-(J3-Pin_1) -> Net-(U2C-+)
- U2 pad 3: Net-(J1-Pin_1) -> Net-(U2A-+)
Routing:
- net Net-(J3-Pin_1): track 61.4 -> 0.00 mm, vias 2 -> 0
- net Net-(U2C-+): track 0.00 -> 60.7 mm, vias 0 -> 2
- net ESP_EN: track 57.5 -> 95.7 mm, vias 2 -> 3
- net Net-(J1-Pin_1): track 28.0 -> 0.00 mm, vias 2 -> 0
- net Net-(U2A-+): track 0.00 -> 27.3 mm, vias 0 -> 2
- net +3.3V: track 396.3 -> 415.2 mm
- net ESP_I0: track 67.0 -> 85.0 mm
- net PHASE3: track 96.3 -> 112.9 mm
- net CAL: track 70.7 -> 83.5 mm
- net Net-(C1-Pad1): track 0.00 -> 11.2 mm
- net Net-(C10-Pad1): track 0.00 -> 11.2 mm
- net GND: track 101.9 -> 112.1 mm, vias 60 -> 64
- net Net-(C2-Pad1): track 4.04 -> 11.3 mm
- net PHASE1: track 75.4 -> 69.2 mm
- net PHASE2: track 85.3 -> 91.1 mm
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Other:
- board size 119.2 x 87.8 mm -> 123.1 x 87.8 mm
- board text added: "EN"
- board text removed: "RESET"

Commit message: -
Routing:
- net GND: vias 64 -> 65
Changed lines of the file:
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@@
+	)
+	(via
+		(at 144.06 50.37)
+		(size 0.6)
+		(drill 0.3)
+		(layers "F.Cu" "B.Cu")
+		(free yes)
+		(net 2)
 	)
 	(via
